Commit message: Use own parameter file to define controller_manager in sim

File: urdf/plugins.urdf.xacro (robot description, xacro)
@@ -1,8 +1,8 @@
 <?xml version="1.0"?>
 <robot xmlns:xacro="http://ros.org/wiki/xacro">
-<xacro:macro name="control" params="namespace controllers_file *remapping:=^">
+<xacro:macro name="control" params="namespace *remapping:=^">
     <gazebo>
         <plugin filename="libgz_ros2_control-system.so" name="gz_ros2_control::GazeboSimROS2ControlPlugin">
-            <parameters>${controllers_file}</parameters>
+            <parameters>$(find duatic_control)/config/controller_manager.yaml</parameters>
             <ros>
                 <namespace>${namespace}</namespace>

Commit message: fix(urdf): add default value for namespace param

File: urdf/plugins.urdf.xacro (robot description, xacro)
@@ -1,5 +1,5 @@
 <?xml version="1.0"?>
 <robot xmlns:xacro="http://ros.org/wiki/xacro">
-<xacro:macro name="control" params="namespace *remapping:=^">
+<xacro:macro name="control" params="namespace:=empty *remapping:=^">
     <gazebo>
         <plugin filename="libgz_ros2_control-system.so" name="gz_ros2_control::GazeboSimROS2ControlPlugin">

Commit message: feat(): added optional remap of topics

File: urdf/plugins.urdf.xacro (robot description, xacro)
@@ -1,5 +1,5 @@
 <?xml version="1.0"?>
 <robot xmlns:xacro="http://ros.org/wiki/xacro">
-<xacro:macro name="control" params="namespace *remapping:=^">
+<xacro:macro name="control" params="namespace:=empty">
     <gazebo>
         <plugin filename="libgz_ros2_control-system.so" name="gz_ros2_control::GazeboSimROS2ControlPlugin">
@@ -11,5 +11,4 @@
                 <remapping>/tf_static:=tf_static</remapping>
                 <remapping>/diagnostics:=diagnostics</remapping>
-                <xacro:insert_block name="remapping" />
             </ros>
         </plugin>

Commit message: update according to reviewers feedback

File: urdf/plugins.urdf.xacro (robot description, xacro)
@@ -1,5 +1,5 @@
 <?xml version="1.0"?>
 <robot xmlns:xacro="http://ros.org/wiki/xacro">
-<xacro:macro name="control" params="namespace:=empty">
+<xacro:macro name="control" params="namespace:=''">
     <gazebo>
         <plugin filename="libgz_ros2_control-system.so" name="gz_ros2_control::GazeboSimROS2ControlPlugin">

Commit message: feat(): added optional remap of topics (#5)
* feat(): added optional remap of topics

* fix(ci): removed check for self-hosted runners

* fix(): added licenses

* feat(): added build status badges

File: urdf/plugins.urdf.xacro (robot description, xacro)
@@ -1,5 +1,13 @@
 <?xml version="1.0"?>
+<!--
+Copyright 2026 Duatic AG
+Redistribution and use in source and binary forms, with or without modification, are permitted provided that the following conditions are met:
+1. Redistributions of source code must retain the above copyright notice, this list of conditions and the following disclaimer.
+2. Redistributions in binary form must reproduce the above copyright notice, this list of conditions and the following disclaimer in the documentation and/or other materials provided with the distribution.
+3. Neither the name of the copyright holder nor the names of its contributors may be used to endorse or promote products derived from this software without specific prior written permission.
+THIS SOFTWARE IS PROVIDED BY THE COPYRIGHT HOLDERS AND CONTRIBUTORS “AS IS” AND ANY EXPRESS OR IMPLIED WARRANTIES, INCLUDING, BUT NOT LIMITED TO, THE IMPLIED WARRANTIES OF MERCHANTABILITY AND FITNESS FOR A PARTICULAR PURPOSE ARE DISCLAIMED. IN NO EVENT SHALL THE COPYRIGHT HOLDER OR CONTRIBUTORS BE LIABLE FOR ANY DIRECT, INDIRECT, INCIDENTAL, SPECIAL, EXEMPLARY, OR CONSEQUENTIAL DAMAGES (INCLUDING, BUT NOT LIMITED TO, PROCUREMENT OF SUBSTITUTE GOODS OR SERVICES; LOSS OF USE, DATA, OR PROFITS; OR BUSINESS INTERRUPTION) HOWEVER CAUSED AND ON ANY THEORY OF LIABILITY, WHETHER IN CONTRACT, STRICT LIABILITY, OR TORT (INCLUDING NEGLIGENCE OR OTHERWISE) ARISING IN ANY WAY OUT OF THE USE OF THIS SOFTWARE, EVEN IF ADVISED OF THE POSSIBILITY OF SUCH DAMAGE.
+-->
 <robot xmlns:xacro="http://ros.org/wiki/xacro">
-<xacro:macro name="control" params="namespace *remapping:=^">
+<xacro:macro name="control" params="namespace:=''">
     <gazebo>
         <plugin filename="libgz_ros2_control-system.so" name="gz_ros2_control::GazeboSimROS2ControlPlugin">
@@ -11,5 +19,4 @@
                 <remapping>/tf_static:=tf_static</remapping>
                 <remapping>/diagnostics:=diagnostics</remapping>
-                <xacro:insert_block name="remapping" />
             </ros>
         </plugin>
